Commit message: trx_s 2軸対応

File: urdf/trx_s.urdf (robot description, URDF)
Before this commit: robot trx_s, 5 links, 4 joints
Links:
- removed link indexbase_link
- removed link indexend_link
- removed link indexmid_link
- removed link thumb_link
- added link base_link1; visual mesh filename=package://trx/urdf/meshes/hand.DAE
- added link base_link2; visual mesh filename=package://trx/urdf/meshes/hand.DAE
- added link indexbase_link1; visual mesh filename=package://trx/urdf/meshes/index_base.DAE
- added link indexbase_link2; visual mesh filename=package://trx/urdf/meshes/index_base.DAE
- added link indexend_link1; visual mesh filename=package://trx/urdf/meshes/index_end.DAE
- added link indexend_link2; visual mesh filename=package://trx/urdf/meshes/index_end.DAE
- added link indexmid_link1; visual mesh filename=package://trx/urdf/meshes/index_mid.DAE
- added link indexmid_link2; visual mesh filename=package://trx/urdf/meshes/index_mid.DAE
- added link thumb_link1; visual mesh filename=package://trx/urdf/meshes/thumb.DAE
- added link thumb_link2; visual mesh filename=package://trx/urdf/meshes/thumb.DAE
- link base_link: geometry 
Joints:
- removed joint indexbase_joint
- removed joint indexend_joint
- removed joint indexmid_joint
- removed joint thumb_joint
- added joint base1_joint: type fixed, parent base_link, child base_link1, origin xyz=0 0.05 0 rpy=0 0 0
- added joint base2_joint: type fixed, parent base_link, child base_link2, origin xyz=0 -0.05 0 rpy=0 0 0
- added joint indexbase_joint1: type revolute, parent base_link1, child indexbase_link1, origin xyz=-0.013 0 0.087 rpy=0 -0 0, axis 0 1 0, limit lower=0.0 upper=1.2 effort=50 velocity=0.5
- added joint indexbase_joint2: type revolute, parent base_link2, child indexbase_link2, origin xyz=-0.013 0 0.087 rpy=0 -0 0, axis 0 1 0, limit lower=0.0 upper=1.2 effort=50 velocity=0.5
- added joint indexend_joint1: type revolute, parent indexmid_link1, child indexend_link1, origin xyz=-0.005 0 0.025 rpy=0 -1.13 0, axis 0 1 0, limit lower=0.0 upper=0.8 effort=50 velocity=0.5
- added joint indexend_joint2: type revolute, parent indexmid_link2, child indexend_link2, origin xyz=-0.005 0 0.025 rpy=0 -1.13 0, axis 0 1 0, limit lower=0.0 upper=0.8 effort=50 velocity=0.5
- added joint indexmid_joint1: type revolute, parent indexbase_link1, child indexmid_link1, origin xyz=0 0 0.045 rpy=0 0.52 0, axis 0 1 0, limit lower=0.0 upper=0.8 effort=50 velocity=0.5
- added joint indexmid_joint2: type revolute, parent indexbase_link2, child indexmid_link2, origin xyz=0 0 0.045 rpy=0 0.52 0, axis 0 1 0, limit lower=0.0 upper=0.8 effort=50 velocity=0.5
- added joint thumb_joint1: type revolute, parent base_link1, child thumb_link1, origin xyz=0.023 0 0.054 rpy=0 -0.08 0, axis 0 1 0, limit lower=-2.0 upper=0.0 effort=50 velocity=10.0
- added joint thumb_joint2: type revolute, parent base_link2, child thumb_link2, origin xyz=0.023 0 0.054 rpy=0 -0.08 0, axis 0 1 0, limit lower=-2.0 upper=0.0 effort=50 velocity=10.0
